Commit message: Added colors to body

File: steer_drive_description/urdf/steer_drive.xacro (robot description, xacro)
@@ -21,5 +21,5 @@
       <mesh filename="package://steer_drive_description/meshes/base_link.stl" scale="0.001 0.001 0.001"/>
     </geometry>
-    <material name="silver"/>
+    <material name="orange"/>
   </visual>
   <collision>
@@ -41,5 +41,5 @@
       <mesh filename="package://steer_drive_description/meshes/lidar_1.stl" scale="0.001 0.001 0.001"/>
     </geometry>
-    <material name="silver"/>
+    <material name="red"/>
   </visual>
   <collision>
@@ -61,5 +61,5 @@
       <mesh filename="package://steer_drive_description/meshes/camera_1.stl" scale="0.001 0.001 0.001"/>
     </geometry>
-    <material name="silver"/>
+    <material name="blue"/>
   </visual>
   <collision>
@@ -81,5 +81,5 @@
       <mesh filename="package://steer_drive_description/meshes/imu_1.stl" scale="0.001 0.001 0.001"/>
     </geometry>
-    <material name="silver"/>
+    <material name="blue"/>
   </visual>
   <collision>
@@ -101,5 +101,5 @@
       <mesh filename="package://steer_drive_description/meshes/arka_hareket_teker_1.stl" scale="0.001 0.001 0.001"/>
     </geometry>
-    <material name="silver"/>
+    <material name="black"/>
   </visual>
   <collision>
@@ -121,5 +121,5 @@
       <mesh filename="package://steer_drive_description/meshes/on_hareket_teker_1.stl" scale="0.001 0.001 0.001"/>
     </geometry>
-    <material name="silver"/>
+    <material name="black"/>
   </visual>
   <collision>
@@ -141,5 +141,5 @@
       <mesh filename="package://steer_drive_description/meshes/arka_donus_teker_1.stl" scale="0.001 0.001 0.001"/>
     </geometry>
-    <material name="silver"/>
+    <material name="green"/>
   </visual>
   <collision>
@@ -161,5 +161,5 @@
       <mesh filename="package://steer_drive_description/meshes/on_donus_teker_1.stl" scale="0.001 0.001 0.001"/>
     </geometry>
-    <material name="silver"/>
+    <material name="orange"/>
   </visual>
   <collision>
@@ -181,5 +181,5 @@
       <mesh filename="package://steer_drive_description/meshes/on_donus_teker_2.stl" scale="0.001 0.001 0.001"/>
     </geometry>
-    <material name="silver"/>
+    <material name="orange"/>
   </visual>
   <collision>
@@ -201,5 +201,5 @@
       <mesh filename="package://steer_drive_description/meshes/on_hareket_teker_2.stl" scale="0.001 0.001 0.001"/>
     </geometry>
-    <material name="silver"/>
+    <material name="black"/>
   </visual>
   <collision>
